Commit message: set rpy to 0 to pass ikfast

File: src/scara_description/robots/mxx_scara.urdf (robot description, URDF)
Before this commit: robot mxx_scara, 5 links, 4 joints
Joints:
- joint joint1: origin xyz=0 0 0.254 rpy=9.3983E-25 2.5634E-20 0.0084538 -> xyz=0 0 0.254 rpy=0 0 0
- joint joint2: origin xyz=0.3 0 -0.003 rpy=1.1025E-21 -2.5499E-20 -0.043209 -> xyz=0.3 0 -0.003 rpy=0 0 0
- joint joint4: origin xyz=0.3 0 -0.11803 rpy=-3.1416 -1.0336E-22 -0.0047866 -> xyz=0.3 0 -0.11803 rpy=-3.14159265359 0 0

Commit message: add tip frame, Translation#AxisAngle needs [1,0,0] Tool Direction, see https://github.com/rdiankov/openrave/issues/596#issuecomment-403673192

File: src/scara_description/robots/mxx_scara.urdf (robot description, URDF)
Before this commit: robot mxx_scara, 5 links, 4 joints
Links:
- added link tip_link
Joints:
- added joint link3_to_tip_link: type fixed, parent link3, child tip_link, origin xyz=0 0 0 rpy=0 1.570796326795 0
